File: hardware/MDD32_Bot/MDD32_Bot.kicad_pcb (KiCad board)
At the start: 4 copper layers, 62 x 28 mm, 66 parts, among them J1 JST_PH, J2 USB_C_Receptacle_USB2.0_16P, J4 Conn_Motor_N20_Encoder, J5 Conn_Motor_N20_Encoder, Q1 AO3401A, Q2 2N7002, Q3 AO3401A, SW1 SW_RESET, SW2 SW_BOOT, SW3 SW_SPDT_SH, U1 ESP32-S3-MINI-1, U2 BQ24072RGT, U3 DRV8833PWPR, U4 AP2114H-3.3, U5 TPS61023DRLR

Commit message: Restructure repo as MDD32 Bot; add firmware and mechanical
Co-authored-by: Cursor <cursoragent@cursor.com>
Parts:
- J2: footprint ESP32_Diff_Drive:USB_C_Receptacle_G-Switch_GT-USB-7010ASV -> MDD32_Bot:USB_C_Receptacle_G-Switch_GT-USB-7010ASV
- L1: footprint ESP32_Diff_Drive:L_Coilcraft_XxL4030 -> MDD32_Bot:L_Coilcraft_XxL4030
- SW3: footprint ESP32_Diff_Drive:SW_SPDT_Shouhan_MSK12C02 -> MDD32_Bot:SW_SPDT_Shouhan_MSK12C02
- U1: footprint ESP32_Diff_Drive:ESP32-S3-MINI-1 -> MDD32_Bot:ESP32-S3-MINI-1
- U2: footprint ESP32_Diff_Drive:VQFN-16-1EP_3x3mm_P0.5mm_EP1.6x1.6mm_ThermalVias -> MDD32_Bot:VQFN-16-1EP_3x3mm_P0.5mm_EP1.6x1.6mm_ThermalVias
- U3: footprint ESP32_Diff_Drive:HTSSOP-16-1EP_4.4x5mm_P0.65mm_EP3.4x5mm_Mask2.66x2.46mm_ThermalVias -> MDD32_Bot:HTSSOP-16-1EP_4.4x5mm_P0.65mm_EP3.4x5mm_Mask2.66x2.46mm_ThermalVias
Other:
- board text added: "MDD32 Bot ${REVISION}"
- board text removed: "ESP32 Diff Drive ${REVISION}"
