File: hardware/MDD32_Bot/MDD32_Bot.kicad_sch (KiCad schematic)
At the start: 66 parts, among them J1 JST_PH, J2 USB_C_Receptacle_USB2.0_16P, J4 Conn_Motor_N20_Encoder, J5 Conn_Motor_N20_Encoder, Q1 AO3401A, Q2 2N7002, Q3 AO3401A, SW1 SW_RESET, SW2 SW_BOOT, SW3 SW_SPDT_SH, U1 ESP32-S3-MINI-1, U2 BQ24072RGT, U3 DRV8833PWPR, U4 AP2114H-3.3, U5 TPS61023DRLR

Commit message: Restructure repo as MDD32 Bot; add firmware and mechanical
Co-authored-by: Cursor <cursoragent@cursor.com>
Parts:
- J2: footprint ESP32_Diff_Drive:USB_C_Receptacle_G-Switch_GT-USB-7010ASV -> MDD32_Bot:USB_C_Receptacle_G-Switch_GT-USB-7010ASV
- J4, J5: symbol ESP32_Diff_Drive:Conn_Motor_N20_Encoder -> MDD32_Bot:Conn_Motor_N20_Encoder
- L1: footprint ESP32_Diff_Drive:L_Coilcraft_XxL4030 -> MDD32_Bot:L_Coilcraft_XxL4030
- SW3: footprint ESP32_Diff_Drive:SW_SPDT_Shouhan_MSK12C02 -> MDD32_Bot:SW_SPDT_Shouhan_MSK12C02; symbol ESP32_Diff_Drive:SW_SPDT_SH -> MDD32_Bot:SW_SPDT_SH
- U1: footprint ESP32_Diff_Drive:ESP32-S3-MINI-1 -> MDD32_Bot:ESP32-S3-MINI-1
- U2: footprint ESP32_Diff_Drive:VQFN-16-1EP_3x3mm_P0.5mm_EP1.6x1.6mm_ThermalVias -> MDD32_Bot:VQFN-16-1EP_3x3mm_P0.5mm_EP1.6x1.6mm_ThermalVias
- U3: footprint ESP32_Diff_Drive:HTSSOP-16-1EP_4.4x5mm_P0.65mm_EP3.4x5mm_Mask2.66x2.46mm_ThermalVias -> MDD32_Bot:HTSSOP-16-1EP_4.4x5mm_P0.65mm_EP3.4x5mm_Mask2.66x2.46mm_ThermalVias; symbol ESP32_Diff_Drive:DRV8833PWPR -> MDD32_Bot:DRV8833PWPR
- U4: symbol ESP32_Diff_Drive:AP2114H-3.3 -> MDD32_Bot:AP2114H-3.3
- U5: symbol ESP32_Diff_Drive:TPS61023DRLR -> MDD32_Bot:TPS61023DRLR
Connections:
- net GND: now also J2.SH (SHIELD); no longer J2.S1 (SHIELD)
- net CS: no longer names the net of U1.21 (IO17)
- net DC: no longer names the net of U1.19 (IO15)
- net LITE: no longer names the net of U1.16 (IO12)
- net MOSI: no longer names the net of U1.18 (IO14)
- net RST: no longer names the net of U1.20 (IO16)
- net SCK: no longer names the net of U1.17 (IO13)
- net SCL: no longer names the net of U1.22 (IO18)
- net SDA: no longer names the net of U1.25 (IO21)
- no-connect marks 24 -> 32
Other:
- title: ESP32 Diff Drive -> MDD32 Bot
